File: Hardware/Mood badge.sch (EAGLE design)
At the start: 9 parts, among them U1 ATMEGA328P_TQFP

Commit message: schematic done
Parts:
- added 487, R21, R22: (no value), LinnesLab-Passives:RESISTOR0603
- added C10, C12: (no value), LinnesLab-Passives:CAPACITOR0603
- added C11, C13, C14, C15, C6: 4.7u, LinnesLab-Passives:CAPACITOR0603
- added C16: 2.2u, LinnesLab-Passives:CAPACITOR0603
- added C17: 1u, LinnesLab-Passives:CAPACITOR0603
- added C18, C7, C8, C9: 100n, LinnesLab-Passives:CAPACITOR0603
- added D1, D2, D3: (no value), LinnesLab-DiscreteSemi:SCHOTTKY-USC
- added FTDI1: FTDI_DEVICE, LinnesLab-Connectors:FTDI_DEVICE
- added J1: AVR_SPI_PROG_3X2NS, LinnesLab-Connectors:AVR_SPI_PROG_3X2NS
- added LED1: (no value), adafruit:SEGMENT_8X8_ROWCATHODEM12A881UR
- added LED2, LED3, LED4, LED5, LED6, LED7, LED8: (no value), LinnesLab-LED:LED0603
- added LIPO1: (no value), LinnesLab-Connectors:JST_2MM_MALE
- added OP1: (no value), LinnesLab-AnalogIC:OP-SINGLEOT
- added R10, R12, R14, R19, R23: 10k, LinnesLab-Passives:RESISTOR0603
- added R11, R13, R15, R16, R17, R18: 1k, LinnesLab-Passives:RESISTOR0603
- added R2, R3, R4, R5, R6, R7, R8, R9: 205, LinnesLab-Passives:RESISTOR0603
- added R20: 12k, LinnesLab-Passives:RESISTOR0603
- added R24: 3.3M, LinnesLab-Passives:RESISTOR0603
- added SW2, SW6: SWITCH.JS202011JXQNUPWARDS, LinnesLab-Switches:SWITCH.JS202011JXQNUPWARDS
- added SW3, SW4, SW5: (no value), LinnesLab-Switches:SPST.KT11P4SM34LFS
- added U$1: ADPS9008, LinnesLab-Sensors:ADPS9008
- added U2: MCP73831.SOT23-5, LinnesLab-Power:MCP73831.SOT23-5
- added USB1: USB.MICRO.PWR-BIGGERPADS, LinnesLab-Connectors:USB.MICRO.PWR-BIGGERPADS
Connections:
- new net N$10: LED1.K6, R7.2
- new net N$11: LED1.K7, R8.2
- new net N$12: LED1.K8, R9.2
- new net N$13: D2.A, SW2.1
- new net N$14: LIPO1.+, SW2.2
- new net N$15: C8.1, LED3.A, R12.2, SW4.B
- new net N$16: C7.1, LED2.A, R10.2, SW3.B
- new net N$17: R10.1, R12.1, R14.1
- new net N$18: LED3.C, R13.2
- new net N$19: LED2.C, R11.2
- new net N$20: C9.1, LED4.A, R14.2, SW5.B
- new net N$21: LED4.C, R15.2
- new net N$22: LED6.C, R17.2
- new net N$23: LED5.C, R16.2
- new net N$24: D3.A, USB1.V+
- new net N$25: 487.2, LED8.C
- new net N$26: LED7.A, R18.1
- new net N$27: R19.2, U2.PROG
- new net N$28: C15.2, C16.1, R23.1
- new net N$29: C16.2, OP1G$1.+IN, R21.1, R22.2
- new net N$30: C13.1, R20.2, U$1.OUT
- new net N$31: C13.2, C14.1, C15.1
- new net N$33: OP1G$1.-IN, R23.2, R24.1
- new net N$4: LED1.K1, R2.2
- new net N$5: LED1.K2, R3.2
- new net N$6: LED1.K3, R4.2
- new net N$7: LED1.K4, R5.2
- new net N$8: LED1.K5, R6.2
- new net N$9: D1.A, FTDI1.VCC
- new net PULSE: OP1G$1.OUT, R24.2
- new net STAT: LED7.C, U2.STAT
- new net VLIPO: C11.1, U2.VBAT
- net DTR: now also FTDI1.DTR
- net GND: now also 487.1, C10.2, C11.2, C12.2, C14.2, C17.1, C18.1, C6.2, C7.2, C8.2, C9.2, FTDI1.CTS, FTDI1.GND, J1.6, LIPO1.-, OP1G$2.V-, R11.1, R13.1, R15.1, R17.1, R19.1, R20.1, R22.1, SW6.1, U$1.GND, U2.VSS, USB1.GND
- net LD1: now also R6.1
- net LD10: now also J1.1, LED1.A4
- net LD11: now also J1.4, LED1.A6
- net LD12: now also R5.1
- net LD13: now also LED1.A1
- net LD14: now also R3.1
- net LD15: now also LED1.A7
- net LD16: now also LED1.A8
- net LD2: now also R8.1
- net LD3: now also LED1.A2
- net LD4: now also LED1.A3
- net LD5: now also R9.1
- net LD6: now also LED1.A5
- net LD7: now also R7.1
- net LD8: now also R4.1
- net LD9: now also J1.3, R2.1
- net MODE: now also LED6.A, R16.1, SW6.2
- net RESET: now also J1.5
- net RXD: now also FTDI1.RXI
- net TXD: now also FTDI1.TXO
- net VCC: now also C10.1, C12.1, C17.2, C18.2, C6.1, D1.C, D2.C, D3.C, J1.2, LED5.A, LED8.A, OP1G$2.V+, R18.2, R21.2, SW3.A, SW4.A, SW5.A, SW6.3, U$1.VCC, U2.VIN
