File: Hardware/Mood badge.brd (EAGLE design)
At the start: 160 x 100 mm, 69 parts, among them J1 AVR_SPI_PROG_3X2NS, SW2 SWITCH.JS202011JXQNUPWARDS, SW6 SWITCH.JS202011JXQNUPWARDS, U1 ATMEGA328P_TQFP, U2 MCP73831.SOT23-5

Commit message: board start
Parts:
- moved C2 1.27 mm to (-6.35, -6.35)
Changed lines of the file:
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@@
 <attribute name="VALUE" x="-8.255" y="-4.445" size="0.7112" layer="27"/>
 </element>
-<element name="C2" library="LinnesLab-Passives" package="C0603" package3d_urn="urn:adsk.eagle:package:15661989/2" value="22p" x="-7.62" y="-6.35" smashed="yes">
-<attribute name="NAME" x="-8.255" y="-5.715" size="0.7112" layer="25"/>
-<attribute name="VALUE" x="-8.255" y="-8.255" size="0.7112" layer="27"/>
+<element name="C2" library="LinnesLab-Passives" package="C0603" package3d_urn="urn:adsk.eagle:package:15661989/2" value="22p" x="-6.35" y="-6.35" smashed="yes">
+<attribute name="NAME" x="-6.985" y="-5.715" size="0.7112" layer="25"/>
+<attribute name="VALUE" x="-6.985" y="-8.255" size="0.7112" layer="27"/>
 </element>
 <element name="Y1" library="LinnesLab-Clocks" package="CA-301" value="" x="-12.7" y="-3.81" smashed="yes">
@@
 <wire x1="-16.18" y1="-23.685" x2="-11.85" y2="-24.13" width="0" layer="19" extent="1-1"/>
 <wire x1="-19.38" y1="-23.685" x2="-16.18" y2="-23.685" width="0" layer="19" extent="1-1"/>
-<wire x1="-6.77" y1="-6.35" x2="-11.85" y2="-20.32" width="0" layer="19" extent="1-1"/>
-<wire x1="-6.77" y1="-2.54" x2="-6.77" y2="-6.35" width="0" layer="19" extent="1-1"/>
+<wire x1="-5.5" y1="-6.35" x2="-11.85" y2="-20.32" width="0" layer="19" extent="1-1"/>
+<wire x1="-6.77" y1="-2.54" x2="-5.5" y2="-6.35" width="0" layer="19" extent="1-1"/>
 <wire x1="-9.3726" y1="7.22" x2="-6.77" y2="-2.54" width="0" layer="19" extent="1-1"/>
 <wire x1="-9.3726" y1="8.82" x2="-9.3726" y2="7.22" width="0" layer="19" extent="1-1"/>
@@
 <contactref element="U1" pad="7"/>
 <contactref element="Y1" pad="2"/>
-<wire x1="-11.176" y1="-3.81" x2="-8.47" y2="-6.35" width="0" layer="19" extent="1-1"/>
+<wire x1="-11.176" y1="-3.81" x2="-7.2" y2="-6.35" width="0" layer="19" extent="1-1"/>
 <wire x1="-9.3726" y1="5.62" x2="-11.176" y2="-3.81" width="0" layer="19" extent="1-1"/>
 </signal>

Commit message: board starting
Parts:
- moved LIPO1 170.2 mm to (33.0, 72.4)
- moved LED1 163.0 mm to (109.2, 39.4)
- moved C6 159.6 mm to (-3.81, 57.1)
- moved C8 159.6 mm to (-8.89, 34.3)
- moved LED3 159.6 mm to (-8.89, 24.1)
- moved R12 159.6 mm to (-5.08, 34.3)
- moved R13 159.6 mm to (-8.89, 29.2)
- moved SW6 159.6 mm to (-6.35, 6.35)
- moved SW2 156.1 mm to (63.5, 12.7)
- moved D2 144.4 mm to (38.1, 10.2)
- moved R2 144.4 mm to (52.1, 48.3)
- moved R3 144.4 mm to (52.1, 44.5)
- moved R4 144.4 mm to (52.1, 40.6)
- moved R5 144.4 mm to (52.1, 36.8)
- moved R6 144.4 mm to (52.1, 33.0)
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Other:
- board size 160 x 100 mm -> 127 x 76.2 mm
